File: CR123A_SAO.kicad_sch (KiCad schematic)
At the start: 18 parts, among them J1 Conn_02x03_Odd_Even, P1 USB_C_Plug_USB2.0, SW1 SW_SPDT_1825232-1, U1 MT3608L

Commit message: ADDING MT2492
Parts:
- added C4, C5: 22μF, Capacitor_SMD:C_0603_1608Metric, symbol sao:C
- added C6: 22nF, Capacitor_SMD:C_0603_1608Metric, symbol sao:C
- added L4: 4.7uH, Swadge_Parts:L_1008_2520Metric, symbol Swadge_Parts:L
- added R4: 36k, symbol sao:R_US
- added R5, R6: 8k, symbol sao:R_US
- added U2: MT2492, Package_TO_SOT_SMD:SOT-23-6, symbol Regulator_Switching:MT3608
- C1, C3, D1, L3, R1, R2, R3, U1: now not fitted; now left out of the parts list
Connections:
- net GND: now also D4.2 (A), C4.2, C5.2, R5.2, U2.2 (GND); no longer BT1.N, BT2.N
- net VCC: now also C4.1, L4.1, R4.1
- net VDC: now also C5.1, R6.1, U2.5 (IN)
- net +9V: now reaches BT1.P
- net +9V: now also D2.1 (K); no longer D4.2 (A)
- net at BT2.P, D2.2 (A): now also BT1.N, D3.1 (K)
- net at BT3.P, D3.2 (A): now also BT2.N, D4.1 (K)
- removed net +3V0: D2.1 (K), D3.1 (K), D4.1 (K), SW1.3 (C)
- new net: R4.2, R5.1, U2.3 (FB)
- new net: R6.2, U2.4 (EN)
- new net: C6.1, L4.2, U2.6 (NC)
- new net: C6.2, U2.1 (BS)
Other:
- moved on the sheet: BT1, BT2, BT3, D2, D3, D4

Commit message: redo layout
Parts:
- R4, R5, R6: footprint (none) -> Resistor_SMD:R_0603_1608Metric
Connections:
- net +9V: now also SW1.3 (C)
Changed lines of the file:
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@@
+	(wire
+		(pts
+			(xy 151.13 68.58) (xy 163.83 68.58)
+		)
+		(stroke
+			(width 0)
+			(type default)
+		)
+	)
 	(wire
 		(pts
@@
 			)
 		)
-		(property "Footprint" ""
+		(property "Footprint" "Resistor_SMD:R_0603_1608Metric"
 			(at 139.446 103.124 90)
 			(effects
@@
 			)
 		)
-		(property "Footprint" ""
+		(property "Footprint" "Resistor_SMD:R_0603_1608Metric"
 			(at 139.446 115.824 90)
 			(effects
@@
 			)
 		)
-		(property "Footprint" ""
+		(property "Footprint" "Resistor_SMD:R_0603_1608Metric"
 			(at 105.156 108.204 90)
 			(effects
@@
 					(unit 1)
 				)
+			)
+		)
+	)
+	(symbol
+		(lib_id "power:+9V")
+		(at 163.83 68.58 0)
+		(unit 1)
+		(exclude_from_sim no)
+		(in_bom yes)
+		(on_board yes)
+		(dnp no)
+		(fields_autoplaced yes)
+		(property "Reference" "#PWR017"
+			(at 163.83 72.39 0)
+			(effects
+				(font
+					(size 1.27 1.27)
+				)
+				(hide yes)
+			)
+		)
+		(property "Value" "+9V"
+			(at 163.83 63.5 0)
+			(effects
+				(font
+					(size 1.27 1.27)
+				)
+			)
+		)
+		(property "Footprint" ""
+			(at 163.83 68.58 0)
+			(effects
+				(font
+					(size 1.27 1.27)
+				)
+				(hide yes)
+			)
+		)
+		(property "Datasheet" ""
+			(at 163.83 68.58 0)
+			(effects
+				(font
+					(size 1.27 1.27)
+				)
+				(hide yes)
+			)
+		)
+		(property "Description" "Power symbol creates a global label with name \"+9V\""
+			(at 163.83 68.58 0)
+			(effects
+				(font
+					(size 1.27 1.27)
+				)
+				(hide yes)
+			)
+		)
+		(pin "1"
+		)
+		(instances
+			(project "CR123A_SAO"
+				(path "/62150cd9-7cc2-47a7-8015-4a50aa20c64e"
+					(reference "#PWR017")
+					(unit 1)
+				)
