File: CR123A_SAO.kicad_pcb (KiCad board)
At the start: 2 copper layers, 68.6 x 96.5 mm, 15 parts, among them J1 Conn_02x03_Odd_Even, P1 USB_C_Plug_USB2.0, SW1 SW_SPDT_1825232-1, U1 MT3608L

Commit message: redo layout
Parts:
- removed C1, C3: 22μF, Capacitor_SMD:C_0603_1608Metric
- removed D1: 1N5817, Diode_THT:D_DO-41_SOD81_P10.16mm_Horizontal
- removed L3: 2.2uH, Swadge_Parts:L_1008_2520Metric
- removed U1: MT3608L, Package_TO_SOT_SMD:SOT-23-6
- added C4: 22μF, Capacitor_SMD:C_0603_1608Metric, F.Cu at (66.5, 53.6)
- added C5: 22μF, Capacitor_SMD:C_0603_1608Metric, F.Cu at (66.5, 56.1)
- added C6: 22nF, Capacitor_SMD:C_0603_1608Metric, F.Cu at (66.5, 58.6)
- added L4: 4.7uH, Swadge_Parts:L_1008_2520Metric, F.Cu at (59.9, 68.5)
- added U2: MT2492, Package_TO_SOT_SMD:SOT-23-6, F.Cu at (60.0, 64.4)
- J1: moved to F.Cu
- moved P1 128.1 mm to (63.2, 38.1), turned to 0 degrees
- moved D3 122.7 mm to (59.3, 21.7), turned to 0 degrees
- moved SW1 118.9 mm to (62.7, 45.5), turned to 0 degrees
- moved D4 111.6 mm to (59.3, 25.9), turned to 0 degrees
- moved D2 108.3 mm to (59.3, 17.4), turned to 0 degrees
- moved BT1 101.0 mm to (33.9, 25.2), turned to 0 degrees
- moved D5 100.2 mm to (59.3, 30.2), turned to 0 degrees
- moved BT3 97.3 mm to (33.9, 64.9), turned to 0 degrees
- moved BT2 97.0 mm to (33.9, 45.1), turned to 0 degrees
- moved J1 77.3 mm to (59.7, 54.6), turned to 0 degrees
Connections:
- BT1 pad N: GND -> Net-(D2-A)
- BT1 pad P: Net-(D4-A) -> +9V
- BT2 pad N: GND -> Net-(D3-A)
- D2 pad 1: +3V0 -> +9V
- D3 pad 1: +3V0 -> Net-(D2-A)
- D4 pad 1: +3V0 -> Net-(D3-A)
- D4 pad 2: Net-(D4-A) -> GND
- SW1 pad 3: +3V0 -> unconnected-(SW1-C-Pad3)
Routing:
- net +3V0: track 60.1 -> 0.00 mm
- net VDC: track 55.5 -> 0.00 mm
- net Net-(D5-A): track 39.3 -> 0.00 mm
- net +5V: track 37.5 -> 0.00 mm
- net VCC: track 20.8 -> 0.00 mm
- net Net-(D3-A): track 8.16 -> 0.00 mm
- net Net-(D4-A): track 7.73 -> 0.00 mm
- net Net-(D1-A): track 7.47 -> 0.00 mm
- net Net-(D2-A): track 7.29 -> 0.00 mm
- net GND: track 1.16 -> 0.00 mm
- removed copper zone on F.Cu, net GND
Other:
- board outline removed

Commit message: sent to jlcpcb
Parts:
- added R4: 36k, Resistor_SMD:R_0603_1608Metric, F.Cu at (57.9, 43.1)
- added R5: 8k, Resistor_SMD:R_0603_1608Metric, F.Cu at (57.9, 46.2)
- added R6: 8k, Resistor_SMD:R_0603_1608Metric, F.Cu at (64.4, 43.8)
- J1: moved to B.Cu
- moved D4 44.5 mm to (43.9, 67.7)
- moved L4 30.9 mm to (61.0, 37.6)
- moved D3 29.9 mm to (38.2, 42.9)
- moved D2 25.6 mm to (43.9, 38.0)
- moved U2 21.6 mm to (61.1, 42.9)
- moved C6 19.1 mm to (61.7, 40.1), turned to 180 degrees
- moved P1 17.9 mm to (77.4, 27.2), turned to 90 degrees
- moved J1 16.3 mm to (74.9, 60.5)
- moved C4 15.7 mm to (55.5, 42.4), turned to 180 degrees
- moved C5 14.7 mm to (65.1, 41.4)
- moved SW1 14.5 mm to (76.7, 41.9), turned to 90 degrees
- moved BT3 14.1 mm to (33.9, 79.0)
- moved BT2 9.55 mm to (33.9, 54.6)
- moved D5 7.17 mm to (65.5, 33.7), turned to 90 degrees
Connections:
- SW1 pad 3: unconnected-(SW1-C-Pad3) -> +9V
Routing:
- net +9V: track 0.00 -> 69.8 mm, vias 0 -> 1
- net Net-(D3-A): track 0.00 -> 63.9 mm
- net Net-(D2-A): track 0.00 -> 59.3 mm
- net VCC: track 0.00 -> 36.3 mm
- net +5V: track 0.00 -> 18.7 mm, vias 0 -> 1
- net VDC: track 0.00 -> 16.5 mm
- net Net-(D5-A): track 0.00 -> 15.3 mm
- net Net-(U2-SW): track 0.00 -> 4.58 mm
- net Net-(U2-FB): track 0.00 -> 3.50 mm
- net Net-(U2-EN): track 0.00 -> 2.45 mm
- net Net-(U2-BS): track 0.00 -> 2.18 mm
- added copper zone on F.Cu, net GND
Other:
- board outline added: 69.5 x 76.6 mm
