File: sao_rtc.kicad_sch (KiCad schematic)
At the start: 42 parts, among them J1 S2B-PH-K-S(LF)(SN), J2 Conn_02x03_Odd_Even, J3 Conn_02x03_Odd_Even, P1 USB_C_Plug_USB2.0, SW1 DPDT, U1 AW32001ECSR, U2 PCF8563DRG, U3 M3410, Y1 32.768 kHz

Commit message: Start of BQ-BMS Swadge SAO
Test Board with BQ24259 BMS chip
WIP
Parts:
- removed C1: 2.2μF, Capacitor_SMD:C_0603_1608Metric, symbol Swadge_Parts:C
- removed C11: 12uF, Capacitor_SMD:C_0603_1608Metric, symbol Swadge_Parts:C
- removed C2, C4, C8: 4.7μF, sao:C_0603_1608Metric, symbol Swadge_Parts:C
- removed C3: 1μF, sao:C_0603_1608Metric, symbol Swadge_Parts:C
- removed C5: C, Capacitor_THT:C_Disc_D3.0mm_W1.6mm_P2.50mm, symbol Device:C
- removed C6: 25pF, C_0603_1608Metric, symbol Swadge_Parts:C
- removed CLK0: TestPoint, TestPoint:TestPoint_Loop_D2.50mm_Drill1.0mm, symbol Connector:TestPoint
- removed D2: 4.3V, Diode_SMD:D_SOD-323_HandSoldering, symbol Device:D_Zener
- removed J1: S2B-PH-K-S(LF)(SN), Connector_PinHeader_2.00mm:PinHeader_1x02_P2.00mm_Horizontal, symbol Swadge_Parts:S2B-PH-K-S(LF)(SN)
- removed L2: 2.2uH, Inductor_SMD:L_0603_1608Metric, symbol Swadge_Parts:L
- removed R1, R3: 5.1kΩ, Resistor_SMD:R_0603_1608Metric, symbol Swadge_Parts:R_US
- removed R2, R5: Ω, Resistor_SMD:R_0603_1608Metric, symbol Swadge_Parts:R_US
- removed R4: 10kΩ, Resistor_SMD:R_0603_1608Metric, symbol Swadge_Parts:R_US
- removed TH1: Thermistor_NTC, Resistor_SMD:R_0603_1608Metric, symbol Swadge_Parts:Thermistor_NTC
- removed U1: AW32001ECSR, Package_CSP:WLCSP-9_1.21x1.22mm_Layout3x3_P0.4mm, symbol Swadge_Parts:AW32001ECSR
- removed U2: PCF8563DRG, Package_SO:SOIC-8_3.9x4.9mm_P1.27mm, symbol Timer_RTC:PCF8563T
- removed Y1: 32.768 kHz, Crystal:Crystal_SMD_3215-2Pin_3.2x1.5mm, symbol Device:Crystal
- added C12: 47nF, sao:C_0603_1608Metric, symbol Swadge_Parts:C
- added C13, C14, C15: 10uF, C_0603_1608Metric, symbol Swadge_Parts:C
- added C16, C17: 22uF, Capacitor_SMD:C_0603_1608Metric, symbol sao:C
- added C5: 4.7μF, sao:C_0603_1608Metric, symbol Swadge_Parts:C
- added D6: D, Diode_SMD:D_SMA, symbol Swadge_Parts:D
- added D7: STAT, LED_SMD:LED_0603_1608Metric, symbol Swadge_Parts:LED
- added H1: 2.54mm Jumper, symbol Auxiliary_Items:Jumper_Shunt
- added JP1: PH2.54-1x3P, Connector_PinHeader_2.54mm:PinHeader_1x03_P2.54mm_Vertical, symbol Jumper:Jumper_3_Open
- added L3: 1uH, Inductor_SMD:L_1008_2520Metric, symbol Swadge_Parts:L
- added R10, R16, R17: 10kΩ, Resistor_SMD:R_0603_1608Metric, symbol Swadge_Parts:R_US
- added R13: 31.6k, Resistor_SMD:R_0603_1608Metric, symbol Swadge_Parts:R_US
- added R14, R15: 22Ω, Resistor_SMD:R_0603_1608Metric, symbol Swadge_Parts:R_US
- added TP1, TP2, TP3, TP4: TestPoint, TestPoint:TestPoint_Loop_D2.60mm_Drill1.4mm_Beaded, symbol Connector:TestPoint
- added U1: BQ24259, Package_DFN_QFN:HVQFN-24-1EP_4x4mm_P0.5mm_EP2.6x2.6mm_ThermalVias, symbol sao:BQ24259
- added U4: NCP1117-3.3_SOT223, Package_TO_SOT_SMD:SOT-223-3_TabPin2, symbol Regulator_Linear:NCP1117-3.3_SOT223
- C7: value (none) -> 10μF; footprint C_0603_1608Metric -> sao:C_0603_1608Metric; Cost @ 2.5k 0.0015 -> (none); Cost100 10 -> (none); LCSC C6119848 -> C85713; now fitted
- D1: Cost @ 2.5k (none) -> 0.4867; Cost100 (none) -> 0.6234; LCSC (none) -> C207262; LCSC Link (none) -> https://www.lcsc.com/product-detail/C207262.html
- D5: value RTC ON -> PGOOD
- R12: value 22Ω -> 5.36k; Cost @ 2.5k 0.0008 -> 0.001; Cost100 10 -> 0.14; LCSC C23345 -> C25973
- SW1: symbol Switch:SW_Slide_DPDT -> Switch:SW_SPDT
Connections:
- net +5V: now also U1.1 (VBUS), U1.24 (VBUS)
- net 3V3: now also C10.1, L1.1, R9.2, C16.1, U4.2 (VO); no longer SW1.1 (A), SW1.5 (B)
- net 3V3 SAO: now also D5.2 (A), D7.2 (A), R16.2, R17.2; no longer SW1.3 (C), SW1.6 (A)
- net BATT+: now also C13.1, D6.2 (A), TP3.1, U1.13 (BAT), U1.14 (BAT)
- net GND: now also C13.2, C14.2, C15.2, C16.2, C17.2, C5.2, JP1.3 (B), R10.1, R13.2, U1.17 (PGND), U1.18 (PGND), U1.2 (PSEL), U1.9 (~{CE}), U1.TP (PAD), U4.1 (GND); no longer R12.1
- net SCL: now also U1.5 (SCL)
- net SDA: now also U1.6 (SDA)
- net VBMS: now also F1.2, SW1.2 (B), C17.1; no longer C9.1, F1.1, R7.2, U3.1 (EN), U3.4 (VIN)
- net PMID: now reaches C7.1
- net PMID: now also U1.23 (PMID)
- net at R12.2: now also JP1.2 (C), R13.1; no longer D5.1 (K)
- removed net VDD: D5.2 (A), SW1.2 (B)
- new net: D7.1 (K), R15.2
- new net: JP1.1 (A), R10.2
- new net: D5.1 (K), R14.2
- new net 3V3_LDO: SW1.1 (A), U4.3 (VI)
- new net 3V3_SW: C9.1, R7.2, SW1.3 (C), U3.1 (EN), U3.4 (VIN)
- new net BMS_INT: TP4.1, U1.7 (INT)
- new net BTST: C12.2, U1.21 (BTST)
- new net REGN: C5.1, U1.22 (REGN)
- new net RTC/CLK0: TP1.1
- new net RTC/V_RTC: D6.1 (K)
- new net RTC/~{INT}: TP2.1
- new net STAT: R15.1, R17.1, U1.4 (STAT)
- new net SW: C12.1, L3.2, U1.19 (SW), U1.20 (SW)
- new net TEMP: R12.1, U1.11 (TS)
- new net VSYS: C14.1, C15.1, F1.1, L3.1, U1.15 (SYS), U1.16 (SYS)
- new net ~{PG}: R14.1, R16.1, U1.3 (~{PG})
- no-connect marks 0 -> 1
Other:
- added sheet Batt Supply (BattSupply.kicad_sch)
- added sheet RTC (Swadge_RTC.kicad_sch)
- note added: "BQ24259 Switches at 1.2Mhz"
- note added: "Pin 12 - QON - Shipping Mode Thing"
- note added: "Pin 2 - PSEL - USB Host Vs Power Brick, Not Important"
- note added: "Pin 21 - BTST - Boot Strap Cap - 47,000pF 10V"
- note added: "Pin 22 - REGN - Driver Supply Cao - 4.7u 10V min"
- note added: "Pin 23 - PMID - Driver Supply Cap - 8.7u 10V min"
- note added: "Pin 8 - OTG - "On-The-Go" USB Boost Charging - Backfeed of Vbatt into Vbus"
- note added: "Pin 9 - ~{CE} - Active Low Charge Enable"
- note added: "RT1/RT2 can be set to values for other NTC curves 5.25k & 31.23k nominal, Rounted to 5.36 & 31.6k since those are the nearest 1% values that I saw in stock"
- note added: "RTC Power Now "Always On" (Downstream of XB7608)"
- note added: "Temperature Test Jumper 10k @ 25C ~27k @ 0C ~5k @ 55C 1-2 For Normal Operation 2-3 For High Temp Trip Remove jumper for Low Temp Trip Install actual 10k NTC between pins 2&3 for real response"
- note removed: "Added a low-pass filter with a 30.8k cutoff frequency to attempt to preempt any noise piped back to the swadge from the crystal. Its a little lower than the crystal frequency because I wanted to use not-weird values for L and C. I added this on the regulator circuit on the SAO to see what happens when it's not present on the identical 3v3 source from the Swadge. This circuit and switch should be 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"
- note removed: "Not sure if we need C7 yet, C5 added for testing"
- note removed: "RTC Power"
- note removed: "Swadge Power"
- moved on the sheet: C10, C9, D1, D3, D4, F1, L1, P1, R11, R6, R7, R8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

Commit message: Complete 1st Draft
First Draft at Schematic Capture and Layout
Parts:
- removed C10, C9: 1μF, Capacitor_SMD:C_0603_1608Metric, symbol Swadge_Parts:C
- removed C12: 47nF, sao:C_0603_1608Metric, symbol Swadge_Parts:C
- removed C13, C14, C15: 10uF, C_0603_1608Metric, symbol Swadge_Parts:C
- removed C5: 4.7μF, sao:C_0603_1608Metric, symbol Swadge_Parts:C
- removed C7: 10μF, sao:C_0603_1608Metric, symbol Swadge_Parts:C
- removed L1: 2.2uH, Inductor_SMD:L_1008_2520Metric, symbol Swadge_Parts:L
- removed L3: 1uH, Inductor_SMD:L_1008_2520Metric, symbol Swadge_Parts:L
- removed R8: 10kΩ, Resistor_SMD:R_0603_1608Metric, symbol Swadge_Parts:R_US
- removed R9: 43kΩ, Resistor_SMD:R_0603_1608Metric, symbol Swadge_Parts:R_US
- removed SW1: DPDT, Button_Switch_SMD:SW_DPDT_CK_JS202011JCQN, symbol Switch:SW_SPDT
- removed U1: BQ24259, Package_DFN_QFN:HVQFN-24-1EP_4x4mm_P0.5mm_EP2.6x2.6mm_ThermalVias, symbol sao:BQ24259
- removed U3: M3410, Package_TO_SOT_SMD:SOT-23-5, symbol Swadge_Parts:M3410
- removed U4: NCP1117-3.3_SOT223, Package_TO_SOT_SMD:SOT-223-3_TabPin2, symbol Regulator_Linear:NCP1117-3.3_SOT223
- removed VMON1: TestPoint, TestPoint:TestPoint_Loop_D2.50mm_Drill1.0mm, symbol Connector:TestPoint
- added C18, C19: 47nF, Capacitor_SMD:C_0603_1608Metric, symbol Swadge_Parts:C
- added L2: 2.2uH, Inductor_SMD:L_1008_2520Metric, symbol Swadge_Parts:L
- added TP5: TP_BMS, TestPoint:TestPoint_Loop_D2.60mm_Drill1.4mm_Beaded, symbol Connector:TestPoint
- added TP6: TP_VMON, TestPoint:TestPoint_Loop_D2.60mm_Drill1.4mm_Beaded, symbol Connector:TestPoint
- added TP7: TP_3V3, TestPoint:TestPoint_Loop_D2.60mm_Drill1.4mm_Beaded, symbol Connector:TestPoint
- J2: value Conn_02x03_Odd_Even -> Connector, In
- J3: value Conn_02x03_Odd_Even -> Connector, Out; footprint Connector_PinHeader_2.54mm:PinHeader_2x03_P2.54mm_Vertical -> sao:PinHeader_2x03_P2.54mm_Vertical_Flipped; LCSC C492420 -> C541853
- TP3: value TestPoint -> TP_BATT
- TP4: value TestPoint -> TP_PGOOD
Connections:
- net 3V3 SAO is gone; now on net 3V3: D4.2 (A), D5.2 (A), D7.2 (A), R16.2, R17.2
- net 3V3_SW is gone; now on net BATT+: R7.2
- net 3V3: now also C18.1, L2.1; no longer C16.1
- net GND: now also C18.2, C19.2
- net at R6.1, R7.1: now also TP6.1
- net BMS_INT renamed BMS/BMS_INT
- net VSYS renamed BMS/VSYS
- net BMS/VSYS: now also TP5.1
- new net 3V3_SAO: C16.1, C19.1, L2.2, TP7.1
- no-connect marks 1 -> 8
Other:
- added sheet 3V3_REG (3V3_REG.kicad_sch)
- added sheet BMS (BMS.kicad_sch)
- note added: "9. RTC Datasheet: https://www.nxp.com/docs/en/data-sheet/PCF8563.pdf"
- note added: "Notes: 1. After power-on, the initial accuracy can be adjusted by testing the output frequency of CLKOUT and adjusting the matching capacitor value of the OSCI pin. If CLKOUT > 32.768kHz, the OSCI capacitor value needs to be increased; if CLKOUT < 32.768kHz, the capacitor value needs to be decreased. 2. Generally, if using a 32.768kHz crystal oscillator with a load capacitor of 12.5pF, approximat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"
- note added: "Pin 3 - ~{PG} - VBUS < Overvoltage Threshold VBUS > 3.8V REGN LDO powered"
- note added: "Test Pi Filter 950khz knee assuming 500mA @ 6.6 ohms / 3.3Vdc 2.2uH 25nF Reusing 2.2uF & the 47nF"
- note added: "The scope has crept up untended by anyone this land is untamed"
- note removed: "9. Datasheet: https://www.nxp.com/docs/en/data-sheet/PCF8563.pdf"
- note removed: "BMS"
- note removed: "BQ24259 Switches at 1.2Mhz"
- note removed: "Notes to self: 1. After power-on, the initial accuracy can be adjusted by testing the output frequency of CLKOUT and adjusting the matching capacitor value of the OSCI pin. If CLKOUT > 32.768kHz, the OSCI capacitor value needs to be increased; if CLKOUT < 32.768kHz, the capacitor value needs to be decreased. 2. Generally, if using a 32.768kHz crystal oscillator with a load capacitor of 12.5pF, ap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"
- note removed: "Pin 12 - QON - Shipping Mode Thing"
- note removed: "Pin 2 - PSEL - USB Host Vs Power Brick, Not Important"
- note removed: "Pin 21 - BTST - Boot Strap Cap - 47,000pF 10V"
- note removed: "Pin 22 - REGN - Driver Supply Cao - 4.7u 10V min"
- note removed: "Pin 23 - PMID - Driver Supply Cap - 8.7u 10V min"
- note removed: "Pin 8 - OTG - "On-The-Go" USB Boost Charging - Backfeed of Vbatt into Vbus"
- note removed: "Pin 9 - ~{CE} - Active Low Charge Enable"
- note removed: "REGULATED 3V3"
- moved on the sheet: C16, C17, D1, D3, D4, D5, D7, J2, J3, JP1, P1, R10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

Commit message: Graphical Cleanup
Just visuals
Other:
- note added: "Test Pi Filter 950khz knee assuming 500mA @ 6.6 ohms / 3.3Vdc 2.2uH 25nF Reusing 2.2uH & the 47nF"
- note removed: "Test Pi Filter 950khz knee assuming 500mA @ 6.6 ohms / 3.3Vdc 2.2uH 25nF Reusing 2.2uF & the 47nF"
- moved on the sheet: C16, C17, C18, C19, D1, D3, D4, D5, D6, D7, F1, J2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
