File: BattSupply.kicad_sch (KiCad schematic)
At the start: 2 parts, among them J1 S2B-PH-K-S(LF)(SN), U5 XB7608AJ

Commit message: Complete 1st Draft
First Draft at Schematic Capture and Layout
Parts:
- U5: footprint (none) -> sao:CPC-5_2.6mmx4mm_P0.53mm
Changed lines of the file:
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@@
 			)
 		)
-		(property "Footprint" ""
+		(property "Footprint" "sao:CPC-5_2.6mmx4mm_P0.53mm"
 			(at 127 111.76 0)
 			(hide yes)
