File: Swadge_RTC.kicad_sch (KiCad schematic)
At the start: 4 parts, among them U2 PCF8563DRG, Y1 32.768 kHz

Commit message: Complete 1st Draft
First Draft at Schematic Capture and Layout
Parts:
- C6: footprint C_0603_1608Metric -> Capacitor_SMD:C_0603_1608Metric
Changed lines of the file:
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@@
 			)
 		)
-		(property "Footprint" "C_0603_1608Metric"
+		(property "Footprint" "Capacitor_SMD:C_0603_1608Metric"
 			(at 102.5652 99.06 0)
 			(hide yes)
