File: 3V3_REG.kicad_sch (KiCad schematic)
At the start: 7 parts, among them U3 MT3410

Commit message: Graphical Cleanup
Just visuals
Other:
- note added: "1.2Mhz Oscillator"
- moved on the sheet: C10, C9, FB1, L1, R8, R9, U3
